Commit message: feat: 선체 크기 조정 기능 추가 (target_length 파라미터화) + 물리 스텝 안정화
kaboat_hull.xacro 신설: WAM-V 선체·엔진·배터리·부력(Surface)·유체동역학
(SimpleHydrodynamics)·추력·센서 장착부를 target_length 파라미터 하나로
비례 스케일(질량 s^3, 관성 s^5)하도록 리팩토링. wamv_kaboat.xacro 는 이를
include 하도록 수정.

배를 4.9m -> 1.1m 로 축소해 검증하는 과정에서 겪은 두 가지 물리 안정성
문제와 해법을 world 설정에 반영:

1. 물리 스텝(max_step_size) 4ms -> 1ms
   작고 가벼워진 선체는 4ms 스텝으로 부력/회전 응답을 안정적으로 적분하지
   못해 "ODE INTERNAL ERROR ... aabbBound" 로 크래시했다 (경계 상태라 몇십
   초 후 지연 크래시하는 경우도 있어 짧은 관찰로는 안정으로 오판하기 쉬웠음).

2. mass_factor 는 절대 1.0 밑으로 낮추지 않기로 결론
   흘수선을 올리려고 질량만 낮추면(관성 유지해도) 부력-질량 진동이 발산해
   같은 크래시가 재현됨을 검증. 관련 내용을 코드 주석 + README §3 에 상세
   기록해 재시도 시 같은 삽질을 반복하지 않도록 함.

부수적으로 발견/확인한 것:
- gain=0(파도 없음)에서도 물 표면이 반짝여 보이는 건 반사광 셰이더
  애니메이션(bumpCoord, amplitude 와 무관)이지 실제 파도가 아님 — 코드
  레벨로 확인, README §4 에 문서화.
- world 의 start_paused=true 때문에 재생 버튼을 눌러야 물리가 시작됨.
- 시뮬 프로세스 종료 시 gz sim 만 죽이면 ros2 launch/parameter_bridge 등
  하위 프로세스가 누적되어 불안정의 숨은 원인이 될 수 있음.
이상 내용을 README §7 문제 해결 섹션으로 정리.

README 전반: 실행 방법 구체화(launch 파일명, headless, 재생 버튼 안내),
선체 크기 조정(§3)/파도 설정(§4) 섹션 신설, ghcr.io 개인 계정 네임스페이스
최초 push 권한 제약 문서화.

Co-Authored-By: Claude Sonnet 5 <noreply@anthropic.com>

File: src/kaboat_sim/urdf/wamv_kaboat.xacro (robot description, xacro)
@@ -1,13 +1,18 @@
 <?xml version="1.0"?>
 <robot xmlns:xacro="http://ros.org/wiki/xacro" name="wamv_kaboat">
-  <xacro:include filename="$(find wamv_gazebo)/urdf/wamv_gazebo.urdf.xacro" />
-  <xacro:include filename="$(find wamv_description)/urdf/thrusters/engine.xacro" />
+  <!-- 크기 조정 가능한 선체 (base_link, 엔진, 배터리, 부력/유체동역학, 추력,
+       상태 퍼블리셔 + 스케일 파라미터 s 를 여기서 정의한다).
+       배 크기는 kaboat_hull.xacro 의 target_length 하나로 조정. -->
+  <xacro:include filename="$(find kaboat_sim)/urdf/kaboat_hull.xacro" />
+  <!-- 위 include 에서 정의된 s(= target_length/base_length)를 그대로 사용해
+       센서 장착부(높이·크기)도 동일 비율로 축소한다. 센서 성능값(라이다 사거리,
+       카메라 FOV/해상도 등)은 물리 치수가 아니므로 스케일하지 않는다. -->
   <link name="cpu_box_link">
     <visual>
-      <geometry><box size="0.4 0.3 0.2"/></geometry>
+      <geometry><box size="${0.4*s} ${0.3*s} ${0.2*s}"/></geometry>
       <material name="cpu_grey"><color rgba="0.6 0.6 0.6 1.0"/></material>
     </visual>
     <collision>
-      <geometry><box size="0.4 0.3 0.2"/></geometry>
+      <geometry><box size="${0.4*s} ${0.3*s} ${0.2*s}"/></geometry>
     </collision>
   </link>
@@ -15,9 +20,9 @@
     <parent link="wamv/base_link"/>
     <child link="cpu_box_link"/>
-    <origin xyz="0.0 0.0 1.3" rpy="0 0 0"/>
+    <origin xyz="0.0 0.0 ${1.3*s}" rpy="0 0 0"/>
   </joint>
   <link name="sensor_pole_link">
     <visual>
-      <geometry><cylinder radius="0.02" length="0.4"/></geometry>
+      <geometry><cylinder radius="${0.02*s}" length="${0.4*s}"/></geometry>
       <material name="pole_black"><color rgba="0.1 0.1 0.1 1.0"/></material>
     </visual>
@@ -26,9 +31,9 @@
     <parent link="cpu_box_link"/>
     <child link="sensor_pole_link"/>
-    <origin xyz="0.1 0.0 0.3" rpy="0 0 0"/>
+    <origin xyz="${0.1*s} 0.0 ${0.3*s}" rpy="0 0 0"/>
   </joint>
   <link name="lidar_link">
     <visual>
-      <geometry><cylinder radius="0.04" length="0.06"/></geometry>
+      <geometry><cylinder radius="${0.04*s}" length="${0.06*s}"/></geometry>
       <material name="lidar_blue"><color rgba="0.0 0.0 0.8 1.0"/></material>
     </visual>
@@ -37,5 +42,5 @@
     <parent link="sensor_pole_link"/>
     <child link="lidar_link"/>
-    <origin xyz="0.0 0.0 0.23" rpy="0 0 0"/>
+    <origin xyz="0.0 0.0 ${0.23*s}" rpy="0 0 0"/>
   </joint>
   <gazebo reference="lidar_link">
@@ -60,5 +65,5 @@
   <link name="camera_link">
     <visual>
-      <geometry><box size="0.03 0.1 0.03"/></geometry>
+      <geometry><box size="${0.03*s} ${0.1*s} ${0.03*s}"/></geometry>
       <material name="cam_black"><color rgba="0.0 0.0 0.0 1.0"/></material>
     </visual>
@@ -67,5 +72,5 @@
     <parent link="sensor_pole_link"/>
     <child link="camera_link"/>
-    <origin xyz="0.12 0.0 0.1" rpy="0 0 0"/>
+    <origin xyz="${0.12*s} 0.0 ${0.1*s}" rpy="0 0 0"/>
   </joint>
   <gazebo reference="camera_link">

Commit message: feat: sensor_drivers 계층 sim 표준 토픽 인터페이스 정비 (IMU·GPS 추가)
- wamv_kaboat.xacro: Gazebo imu(100Hz)/navsat(10Hz) 센서 추가
  (world 에 imu-system·NavSat 플러그인 + spherical_coordinates 이미 존재)
- bridge_config.yaml: 전 센서를 node_structure v5 표준 이름으로 정규화
  (/lidar/scan→/scan, /camera/depth/image→/camera/image_raw,
   /camera/depth/points→/depth/points, +/imu/data, /navsat→/gps/fix)
- simulation.launch.py: 인라인 @ 브리지 → config_file 방식
  (이름 리매핑은 인라인 문법 불가, config 파일만 ros명≠gz명 지원)
- README: §5 센서 토픽 인터페이스 표 + §6 현재 브랜치 안내 추가

sim 에서는 Gazebo 가 sensor_msgs 로 발행하므로 UART 파싱 불필요.
실물 전환 시 각 드라이버가 동일 표준 토픽으로 발행하면 상위 노드 변경 없음.

Co-Authored-By: Claude Opus 4.8 <noreply@anthropic.com>

File: src/kaboat_sim/urdf/wamv_kaboat.xacro (robot description, xacro)
@@ -93,3 +93,46 @@
     </sensor>
   </gazebo>
+  <!-- IMU (실물: EBIMU-9DOFv5-R3, UART). sim 에서는 Gazebo imu 센서가
+       sensor_msgs/Imu 로 바로 발행하므로 UART 파싱 불필요. 실물 전환 시
+       이 노드만 UART 드라이버로 교체하고 토픽 인터페이스(/imu/data)는 유지. -->
+  <link name="imu_link">
+    <visual>
+      <geometry><box size="${0.02*s} ${0.02*s} ${0.01*s}"/></geometry>
+      <material name="imu_green"><color rgba="0.0 0.6 0.2 1.0"/></material>
+    </visual>
+  </link>
+  <joint name="imu_joint" type="fixed">
+    <parent link="wamv/base_link"/>
+    <child link="imu_link"/>
+    <origin xyz="0.0 0.0 ${0.2*s}" rpy="0 0 0"/>
+  </joint>
+  <gazebo reference="imu_link">
+    <sensor name="imu_sensor" type="imu">
+      <always_on>true</always_on>
+      <update_rate>100</update_rate>
+      <topic>/imu/data</topic>
+      <gz_frame_id>imu_link</gz_frame_id>
+    </sensor>
+  </gazebo>
+  <!-- GPS (실물: 기종 미정, NMEA/serial 예상). sim 에서는 Gazebo navsat 센서가
+       sensor_msgs/NavSatFix 로 발행. world 의 spherical_coordinates 원점 기준. -->
+  <link name="gps_link">
+    <visual>
+      <geometry><cylinder radius="${0.02*s}" length="${0.02*s}"/></geometry>
+      <material name="gps_grey"><color rgba="0.4 0.4 0.4 1.0"/></material>
+    </visual>
+  </link>
+  <joint name="gps_joint" type="fixed">
+    <parent link="sensor_pole_link"/>
+    <child link="gps_link"/>
+    <origin xyz="0.0 0.0 ${0.26*s}" rpy="0 0 0"/>
+  </joint>
+  <gazebo reference="gps_link">
+    <sensor name="navsat_sensor" type="navsat">
+      <always_on>true</always_on>
+      <update_rate>10</update_rate>
+      <topic>/navsat</topic>
+      <gz_frame_id>gps_link</gz_frame_id>
+    </sensor>
+  </gazebo>
 </robot>
